File: the superior KiCad/BattleBits_V4.kicad_sch (KiCad schematic)
At the start: 107 parts

Commit message: kicad
Connections:
- net GND: no longer C2.2, C4.1, C6.1, IC1.14 (VDD), IC10.2 (VOUT), IC11.10 (-IN), IC11.3 (V+), IC11.4 (-IN), IC11.6 (-IN), IC11.8 (-IN), IC12.3 (V+), IC2.9 (CD+), IC3.14 (VDD), IC4.9 (CD+), IC5.9 (CD+), IC6.9 (CD+), IC7.9 (CD+), IC8.3 (VCC@2), IC9.3 (VCC@2), JP1.2, JP2.2, PH1.1, PH2.1, PH3.1, PH4.1, PH5.1, PH6.1, PH7.1, PH8.1, R12.1, R17.1, R18.1, R18.2, R8.1, R9.1, SV10.1, SV10.6, SV11.1, SV11.6, SV12.1, SV12.6, SV14.1, SV14.2, SV14.3, SV15.1, SV15.2, SV15.3, SV9.1, SV9.6, U$10.10, U$10.5, U$11.10, U$11.5, U$19.10, U$19.5, U$20.10, U$20.5, U$3.10, U$3.5, U$4.10, U$4.5, U$5.10, U$5.5, U$6.10, U$6.5, U$9.10, U$9.5
- new net: IC11.10 (-IN), IC11.4 (-IN), IC11.6 (-IN), IC11.8 (-IN), R17.1, R18.2
- new net VDD: C2.2, C4.1, C6.1, IC1.14 (VDD), IC10.2 (VOUT), IC11.3 (V+), IC12.3 (V+), IC2.9 (CD+), IC3.14 (VDD), IC4.9 (CD+), IC5.9 (CD+), IC6.9 (CD+), IC7.9 (CD+), IC8.3 (VCC@2), IC9.3 (VCC@2), JP1.2, JP2.2, PH1.1, PH2.1, PH3.1, PH4.1, PH5.1, PH6.1, PH7.1, PH8.1, R12.1, R18.1, R8.1, R9.1, SV10.1, SV10.6, SV11.1, SV11.6, SV12.1, SV12.6, SV14.1, SV14.2, SV14.3, SV15.1, SV15.2, SV15.3, SV9.1, SV9.6, U$10.10, U$10.5, U$11.10, U$11.5, U$19.10, U$19.5, U$20.10, U$20.5, U$3.10, U$3.5, U$4.10, U$4.5, U$5.10, U$5.5, U$6.10, U$6.5, U$9.10, U$9.5
Changed lines of the file:
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@@
   (junction (at 223.52 241.3) (diameter 0) (color 0 0 0 0)
   )
-  (junction (at 382.27 116.84) (diameter 0) (color 0 0 0 0)
-  )
   (junction (at 220.98 182.88) (diameter 0) (color 0 0 0 0)
   )
@@
   (junction (at 403.86 71.12) (diameter 0) (color 0 0 0 0)
   )
-  (junction (at 403.86 109.22) (diameter 0) (color 0 0 0 0)
-  )
   (junction (at 223.52 231.14) (diameter 0) (color 0 0 0 0)
   )
@@
   (junction (at 220.98 180.34) (diameter 0) (color 0 0 0 0)
   )
-  (junction (at 382.27 109.22) (diameter 0) (color 0 0 0 0)
-  )
   (junction (at 223.52 266.7) (diameter 0) (color 0 0 0 0)
   )
   (junction (at 396.24 116.84) (diameter 0) (color 0 0 0 0)
   )
-  (junction (at 410.21 116.84) (diameter 0) (color 0 0 0 0)
-  )
   (junction (at 223.52 236.22) (diameter 0) (color 0 0 0 0)
   )
@@
     (stroke (width 0) (type default) (color 0 0 0 0))
   )
-  (wire (pts (xy 554.99 116.84) (xy 554.99 132.08))
+  (wire (pts (xy 554.99 116.84) (xy 554.99 113.03))
     (stroke (width 0) (type default) (color 0 0 0 0))
   )
@@
     (stroke (width 0) (type default) (color 0 0 0 0))
   )
-  (wire (pts (xy 382.27 109.22) (xy 382.27 116.84))
-    (stroke (width 0) (type default) (color 0 0 0 0))
-  )
   (wire (pts (xy 144.78 182.88) (xy 142.24 182.88))
     (stroke (width 0) (type default) (color 0 0 0 0))
@@
     (stroke (width 0) (type default) (color 0 0 0 0))
   )
-  (wire (pts (xy 601.98 132.08) (xy 601.98 119.38))
+  (wire (pts (xy 601.98 113.03) (xy 601.98 119.38))
     (stroke (width 0) (type default) (color 0 0 0 0))
   )
@@
     (stroke (width 0) (type default) (color 0 0 0 0))
   )
-  (wire (pts (xy 408.94 116.84) (xy 410.21 116.84))
+  (wire (pts (xy 408.94 116.84) (xy 554.99 116.84))
     (stroke (width 0) (type default) (color 0 0 0 0))
   )
@@
     (stroke (width 0) (type default) (color 0 0 0 0))
   )
-  (wire (pts (xy 248.92 63.5) (xy 248.92 60.96))
+  (wire (pts (xy 248.92 59.69) (xy 248.92 63.5))
     (stroke (width 0) (type default) (color 0 0 0 0))
   )
@@
     (stroke (width 0) (type default) (color 0 0 0 0))
   )
-  (wire (pts (xy 355.6 109.22) (xy 382.27 109.22))
+  (wire (pts (xy 355.6 109.22) (xy 396.24 109.22))
     (stroke (width 0) (type default) (color 0 0 0 0))
   )
@@
     (stroke (width 0) (type default) (color 0 0 0 0))
   )
-  (wire (pts (xy 574.04 119.38) (xy 568.96 119.38))
+  (wire (pts (xy 574.04 119.38) (xy 567.69 119.38))
     (stroke (width 0) (type default) (color 0 0 0 0))
   )
@@
     (stroke (width 0) (type default) (color 0 0 0 0))
   )
-  (wire (pts (xy 554.99 132.08) (xy 601.98 132.08))
+  (wire (pts (xy 554.99 113.03) (xy 601.98 113.03))
     (stroke (width 0) (type default) (color 0 0 0 0))
   )
@@
     (stroke (width 0) (type default) (color 0 0 0 0))
   )
-  (wire (pts (xy 410.21 109.22) (xy 403.86 109.22))
-    (stroke (width 0) (type default) (color 0 0 0 0))
-  )
   (wire (pts (xy 160.02 284.48) (xy 162.56 284.48))
     (stroke (width 0) (type default) (color 0 0 0 0))
@@
     (stroke (width 0) (type default) (color 0 0 0 0))
   )
-  (wire (pts (xy 410.21 116.84) (xy 554.99 116.84))
-    (stroke (width 0) (type default) (color 0 0 0 0))
-  )
   (wire (pts (xy 271.78 93.98) (xy 274.32 93.98))
     (stroke (width 0) (type default) (color 0 0 0 0))
@@
     (stroke (width 0) (type default) (color 0 0 0 0))
   )
-  (wire (pts (xy 568.96 124.46) (xy 568.96 119.38))
+  (wire (pts (xy 567.69 124.46) (xy 567.69 119.38))
     (stroke (width 0) (type default) (color 0 0 0 0))
   )
@@
     (stroke (width 0) (type default) (color 0 0 0 0))
   )
-  (wire (pts (xy 375.92 124.46) (xy 568.96 124.46))
+  (wire (pts (xy 375.92 124.46) (xy 567.69 124.46))
     (stroke (width 0) (type default) (color 0 0 0 0))
   )
@@
     (stroke (width 0) (type default) (color 0 0 0 0))
   )
-  (wire (pts (xy 410.21 116.84) (xy 410.21 109.22))
-    (stroke (width 0) (type default) (color 0 0 0 0))
-  )
   (wire (pts (xy 220.98 177.8) (xy 276.86 177.8))
     (stroke (width 0) (type default) (color 0 0 0 0))
@@
   )
   (wire (pts (xy 429.26 223.52) (xy 439.42 223.52))
-    (stroke (width 0) (type default) (color 0 0 0 0))
-  )
-  (wire (pts (xy 382.27 109.22) (xy 396.24 109.22))
     (stroke (width 0) (type default) (color 0 0 0 0))
   )
@@
     (effects (font (size 0.889 0.889)) (justify left bottom))
   )
-  (label "GND" (at 568.96 119.38 180)
+  (label "GND" (at 567.69 119.38 180)
     (effects (font (size 0.889 0.889)) (justify right bottom))
   )
@@
     (effects (font (size 0.889 0.889)) (justify right bottom))
   )
-  (label "GND" (at 248.92 60.96 90)
-    (effects (font (size 0.889 0.889)) (justify left bottom))
-  )
+  (label "GND" (at 248.92 59.69 90)
+    (effects (font (size 0.889 0.889)) (justify left bottom))
+  )

Commit message: -
Parts:
- C1, C2, C3, C4, C5, C6: value (none) -> 10uF; footprint (none) -> BattleBits_V4:C3216
- D1, D10, D11, D12, D15, D16, D17, D18, D19, D2, D20, D21, D22, D23, D24, D25, D26, D3, D4, D5, D6, D7, D8, D9: value (none) -> LED1206; footprint (none) -> BattleBits_V4:LED-1206
- D13: value (none) -> DIODESMA; footprint (none) -> BattleBits_V4:SMADIODE
- IC1, IC3: value (none) -> 4001N; footprint (none) -> BattleBits_V4:DIL14
- IC10: value (none) -> REG1117; footprint (none) -> BattleBits_V4:SOT223
- IC11, IC12: value (none) -> LM2901D; footprint (none) -> BattleBits_V4:SO14
- IC2, IC4, IC5, IC6, IC7: value (none) -> ULN2004AD; footprint (none) -> BattleBits_V4:SO16
- IC8, IC9: value (none) -> BD623F; footprint (none) -> BattleBits_V4:SOP8
- JP1, JP2, JP8: value (none) -> PINHD-1X2; footprint (none) -> BattleBits_V4:1X02
- LED_A0, LED_B0, LED_C0, LED_D0, LED_E0, LED_F0, LED_G0, LED_H0: value (none) -> LED5MM; footprint (none) -> BattleBits_V4:LED5MM
- PH1, PH2, PH3, PH4, PH5, PH6, PH7, PH8: value (none) -> ?1060V; footprint (none) -> BattleBits_V4:TO-5_V10
- R1, R10, R11, R14, R2, R3, R4, R5, R6, R7: value (none) -> 3362P-1-103LF; footprint (none) -> BattleBits_V4:3362P-1-103LF
- R12, R13: value (none) -> 5K, 1%; footprint (none) -> BattleBits_V4:R3216
- R15, R16: value (none) -> 20K, 1%; footprint (none) -> BattleBits_V4:R3216
- R8, R9: value (none) -> 30k; footprint (none) -> BattleBits_V4:R3216
- SV1, SV10, SV11, SV12, SV13, SV14, SV15, SV2, SV3, SV4, SV5, SV6, SV7, SV8, SV9: value (none) -> FE06-1; footprint (none) -> BattleBits_V4:FE06
- U$1, U$2: value (none) -> MOTOR; footprint (none) -> BattleBits_V4:GEARMOTOR
- U$10, U$11, U$19, U$20, U$3, U$5, U$6, U$9: value (none) -> 10K; footprint (none) -> BattleBits_V4:EXBA
- U$4: value (none) -> 330; footprint (none) -> BattleBits_V4:EXBA
- U$7: value (none) -> SLIDE_SWITCH; footprint (none) -> BattleBits_V4:SLIDE_SWITCH
